File: LampSmoke/FogMachineTimer_revB/FogMachineTimer_revB.sch (EAGLE design)
At the start: 10 parts, among them J1 M20-9980346, J2 CUI_PJ-037ACUI_PJ-037A_0_0

Commit message: added code and power reg
Parts:
- added C2: 0.33uF, SparkFun-Capacitors:0.1UF-0603-25V-5%
- added LM7805: 7805DT, adafruit:7805DT
- R1: value 1k -> 1k5
- R2: value 56R -> 1k5
Connections:
- removed net U1_P6: R1.1, RELAY.4
- new net N$3: R1.2, RELAY.3
- new net VIN: C2.2, J2.1, LM7805.VI
- net GND: now also C2.1, LM7805.GND
- net PB0: now also R1.1; no longer RELAY.3
- net SW_POS: now also RELAY.4; no longer R1.2
- net VCC: now also LM7805.VO; no longer J2.1
Other:
- moved on the sheet: C1, R1
Changed lines of the file:
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@@
 <part name="J2" library="NickParts" library_urn="urn:adsk.eagle:library:4753178" deviceset="CUI_PJ-037A" device="CUI_PJ-037A_0_0" package3d_urn="urn:adsk.eagle:package:4865637/3"/>
 <part name="J3" library="SparkFun-Connectors" library_urn="urn:adsk.eagle:library:513" deviceset="CONN_02" device="" package3d_urn="urn:adsk.eagle:package:38039/1"/>
-<part name="R1" library="SparkFun-Resistors" library_urn="urn:adsk.eagle:library:532" deviceset="1KOHM" device="-0603-1/10W-1%" package3d_urn="urn:adsk.eagle:package:39650/1" value="1k"/>
+<part name="R1" library="SparkFun-Resistors" library_urn="urn:adsk.eagle:library:532" deviceset="1KOHM" device="-0603-1/10W-1%" package3d_urn="urn:adsk.eagle:package:39650/1" value="1k5"/>
 <part name="D1" library="SparkFun-LED" library_urn="urn:adsk.eagle:library:529" deviceset="LED" device="1206" package3d_urn="urn:adsk.eagle:package:39352/1"/>
-<part name="R2" library="SparkFun-Resistors" library_urn="urn:adsk.eagle:library:532" deviceset="1KOHM" device="-0603-1/10W-1%" package3d_urn="urn:adsk.eagle:package:39650/1" value="56R"/>
+<part name="R2" library="SparkFun-Resistors" library_urn="urn:adsk.eagle:library:532" deviceset="1KOHM" device="-0603-1/10W-1%" package3d_urn="urn:adsk.eagle:package:39650/1" value="1k5"/>
 <part name="C1" library="SparkFun-Capacitors" library_urn="urn:adsk.eagle:library:510" deviceset="0.1UF" device="-0603-25V-5%" package3d_urn="urn:adsk.eagle:package:37414/1" value="0.1uF"/>
 <part name="RELAY" library="NickParts" library_urn="urn:adsk.eagle:library:4753178" deviceset="HE3621A0510" device="" package3d_urn="urn:adsk.eagle:package:13183713/2"/>
 <part name="D2" library="SparkFun-LED" library_urn="urn:adsk.eagle:library:529" deviceset="LED" device="1206" package3d_urn="urn:adsk.eagle:package:39352/1"/>
+<part name="LM7805" library="adafruit" library_urn="urn:adsk.eagle:library:420" deviceset="78*" device="DT" package3d_urn="urn:adsk.eagle:package:6240672/1" technology="05"/>
+<part name="C2" library="SparkFun-Capacitors" library_urn="urn:adsk.eagle:library:510" deviceset="0.1UF" device="-0603-25V-5%" package3d_urn="urn:adsk.eagle:package:37414/1" value="0.33uF"/>
 </parts>
 <sheets>
@@
 <attribute name="NAME" x="30.48" y="102.108" size="1.778" layer="95" font="vector"/>
 </instance>
-<instance part="R1" gate="G$1" x="66.04" y="134.62" smashed="yes">
-<attribute name="NAME" x="66.04" y="136.144" size="1.778" layer="95" font="vector" align="bottom-center"/>
-<attribute name="VALUE" x="66.04" y="133.096" size="1.778" layer="96" font="vector" align="top-center"/>
+<instance part="R1" gate="G$1" x="17.78" y="134.62" smashed="yes">
+<attribute name="NAME" x="17.78" y="136.144" size="1.778" layer="95" font="vector" align="bottom-center"/>
+<attribute name="VALUE" x="17.78" y="133.096" size="1.778" layer="96" font="vector" align="top-center"/>
 </instance>
 <instance part="D1" gate="G$1" x="101.6" y="99.06" smashed="yes" rot="R270">
@@
 <attribute name="VALUE" x="121.92" y="97.536" size="1.778" layer="96" font="vector" align="top-center"/>
 </instance>
-<instance part="C1" gate="G$1" x="137.16" y="127" smashed="yes" rot="R180">
-<attribute name="NAME" x="135.636" y="124.079" size="1.778" layer="95" font="vector" rot="R180"/>
-<attribute name="VALUE" x="135.636" y="129.159" size="1.778" layer="96" font="vector" rot="R180"/>
+<instance part="C1" gate="G$1" x="152.4" y="142.24" smashed="yes" rot="R180">
+<attribute name="NAME" x="150.876" y="139.319" size="1.778" layer="95" font="vector" rot="R180"/>
+<attribute name="VALUE" x="150.876" y="144.399" size="1.778" layer="96" font="vector" rot="R180"/>
 </instance>
 <instance part="RELAY" gate="G$1" x="38.1" y="129.54" smashed="yes" rot="R90"/>
@@
 <attribute name="NAME" x="107.188" y="102.489" size="1.778" layer="95" font="vector"/>
 <attribute name="VALUE" x="107.188" y="97.155" size="1.778" layer="96" font="vector" align="top-left"/>
+</instance>
+<instance part="LM7805" gate="A1" x="137.16" y="154.94" smashed="yes">
+<attribute name="NAME" x="129.54" y="160.655" size="1.778" layer="95"/>
+<attribute name="VALUE" x="129.54" y="158.115" size="1.778" layer="96"/>
+</instance>
+<instance part="C2" gate="G$1" x="127" y="142.24" smashed="yes" rot="R180">
+<attribute name="NAME" x="125.476" y="139.319" size="1.778" layer="95" font="vector" rot="R180"/>
+<attribute name="VALUE" x="125.476" y="144.399" size="1.778" layer="96" font="vector" rot="R180"/>
 </instance>
 </instances>
@@
 <segment>
 <pinref part="J2" gate="G$0" pin="2"/>
-<wire x1="109.22" y1="124.46" x2="114.3" y2="124.46" width="0.1524" layer="91"/>
 <label x="114.3" y="124.46" size="1.778" layer="95" xref="yes"/>
 <pinref part="C1" gate="G$1" pin="1"/>
-<wire x1="137.16" y1="121.92" x2="114.3" y2="121.92" width="0.1524" layer="91"/>
-<wire x1="114.3" y1="121.92" x2="114.3" y2="124.46" width="0.1524" layer="91"/>
+<wire x1="152.4" y1="137.16" x2="152.4" y2="124.46" width="0.1524" layer="91"/>
+<wire x1="152.4" y1="124.46" x2="137.16" y2="124.46" width="0.1524" layer="91"/>
+<pinref part="LM7805" gate="A1" pin="GND"/>
+<wire x1="137.16" y1="124.46" x2="109.22" y2="124.46" width="0.1524" layer="91"/>
+<wire x1="137.16" y1="147.32" x2="137.16" y2="137.16" width="0.1524" layer="91"/>
+<pinref part="C2" gate="G$1" pin="1"/>
+<wire x1="127" y1="137.16" x2="137.16" y2="137.16" width="0.1524" layer="91"/>
+<wire x1="137.16" y1="137.16" x2="137.16" y2="124.46" width="0.1524" layer="91"/>
+<junction x="137.16" y="137.16"/>
+<junction x="137.16" y="124.46"/>
 </segment>
 </net>
@@
 </segment>
 <segment>
-<pinref part="J2" gate="G$0" pin="1"/>
-<wire x1="109.22" y1="129.54" x2="114.3" y2="129.54" width="0.1524" layer="91"/>
-<label x="114.3" y="129.54" size="1.778" layer="95" xref="yes"/>
+<pinref part="LM7805" gate="A1" pin="VO"/>
+<wire x1="152.4" y1="154.94" x2="147.32" y2="154.94" width="0.1524" layer="91"/>
 <pinref part="C1" gate="G$1" pin="2"/>
-<wire x1="137.16" y1="129.54" x2="137.16" y2="134.62" width="0.1524" layer="91"/>
-<wire x1="137.16" y1="134.62" x2="114.3" y2="134.62" width="0.1524" layer="91"/>
-<wire x1="114.3" y1="134.62" x2="114.3" y2="129.54" width="0.1524" layer="91"/>
+<wire x1="152.4" y1="154.94" x2="152.4" y2="144.78" width="0.1524" layer="91"/>
+<label x="152.4" y="154.94" size="1.778" layer="95" xref="yes"/>
 </segment>
 </net>
@@
 </segment>
 <segment>
-<label x="17.78" y="134.62" size="1.778" layer="95" rot="R180" xref="yes"/>
-<wire x1="17.78" y1="134.62" x2="27.94" y2="134.62" width="0.1524" layer="91"/>
-<wire x1="27.94" y1="134.62" x2="27.94" y2="132.08" width="0.1524" layer="91"/>
-<pinref part="RELAY" gate="G$1" pin="3"/>
-<wire x1="27.94" y1="132.08" x2="35.56" y2="132.08" width="0.1524" layer="91"/>
+<pinref part="R1" gate="G$1" pin="1"/>
+<wire x1="12.7" y1="134.62" x2="5.08" y2="134.62" width="0.1524" layer="91"/>
+<label x="5.08" y="134.62" size="1.778" layer="95" rot="R180" xref="yes"/>
 </segment>
 </net>
@@
 </segment>
 <segment>
-<pinref part="R1" gate="G$1" pin="2"/>
-<wire x1="71.12" y1="134.62" x2="76.2" y2="134.62" width="0.1524" layer="91"/>
-<label x="76.2" y="134.62" size="1.778" layer="95" xref="yes"/>
-</segment>
-</net>
-<net name="U1_P6" class="0">
-<segment>
-<pinref part="R1" gate="G$1" pin="1"/>
 <pinref part="RELAY" gate="G$1" pin="4"/>
 <wire x1="35.56" y1="137.16" x2="35.56" y2="139.7" width="0.1524" layer="91"/>
 <wire x1="35.56" y1="139.7" x2="43.18" y2="139.7" width="0.1524" layer="91"/>
 <wire x1="43.18" y1="139.7" x2="43.18" y2="134.62" width="0.1524" layer="91"/>
-<wire x1="43.18" y1="134.62" x2="60.96" y2="134.62" width="0.1524" layer="91"/>
+<wire x1="43.18" y1="134.62" x2="58.42" y2="134.62" width="0.1524" layer="91"/>
+<label x="58.42" y="134.62" size="1.778" layer="95" xref="yes"/>
 </segment>
 </net>
@@
 </segment>
 </net>
+<net name="N$3" class="0">
+<segment>
+<pinref part="R1" gate="G$1" pin="2"/>
+<wire x1="22.86" y1="134.62" x2="22.86" y2="132.08" width="0.1524" layer="91"/>
+<wire x1="22.86" y1="132.08" x2="35.56" y2="132.08" width="0.1524" layer="91"/>
+<pinref part="RELAY" gate="G$1" pin="3"/>
+</segment>
+</net>
+<net name="VIN" class="0">
+<segment>
+<pinref part="LM7805" gate="A1" pin="VI"/>
+<wire x1="127" y1="154.94" x2="109.22" y2="154.94" width="0.1524" layer="91"/>
+<pinref part="J2" gate="G$0" pin="1"/>
+<wire x1="109.22" y1="154.94" x2="109.22" y2="129.54" width="0.1524" layer="91"/>
+<label x="109.22" y="142.24" size="1.778" layer="95" xref="yes"/>
+<pinref part="C2" gate="G$1" pin="2"/>
+<wire x1="127" y1="144.78" x2="127" y2="154.94" width="0.1524" layer="91"/>
+<junction x="127" y="154.94"/>
+</segment>
+</net>
